File: pcb/ekomigacz.brd (EAGLE design)
At the start: 26.7 x 38.7 mm, 9 parts, among them X1 USB-A-H

Commit message: Update
Parts:
- moved JP2 4.57 mm to (22.2, 15.4)
Routing:
- net N$7: track 11.4 -> 6.86 mm
- net N$6: track 4.86 -> 2.86 mm
Changed lines of the file:
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@@
 <?xml version="1.0" encoding="utf-8"?>
 <!DOCTYPE eagle SYSTEM "eagle.dtd">
-<eagle version="9.3.2">
+<eagle version="9.4.0">
 <drawing>
 <settings>
@@
 <layer number="43" name="vRestrict" color="2" fill="10" visible="yes" active="yes"/>
 <layer number="44" name="Drills" color="7" fill="1" visible="no" active="yes"/>
-<layer number="45" name="Holes" color="7" fill="1" visible="no" active="yes"/>
+<layer number="45" name="Holes" color="7" fill="1" visible="yes" active="yes"/>
 <layer number="46" name="Milling" color="3" fill="1" visible="no" active="yes"/>
 <layer number="47" name="Measures" color="7" fill="1" visible="no" active="yes"/>
@@
 </layers>
 <board>
-<fusionsync huburn="a.cGVyc29uYWw6dWUyYzZlMjc0" projecturn="a.cGVyc29uYWw6dWUyYzZlMjc0IzIwMTkwNDA3MTg2OTg1MjI2" f3durn="urn:adsk.wipprod:dm.lineage:er7lF2gcRpaTRLaYGySQig" pcbguid="eab0e8ed-70a1-480c-828d-d798c72a6244" lastpulledtime="" lastsyncedchangeguid="af343b81-1785-c379-00e7-872bfe1e5a25"/>
+<fusionsync huburn="a.cGVyc29uYWw6dWUyYzZlMjc0" projecturn="a.cGVyc29uYWw6dWUyYzZlMjc0IzIwMTkwNDA3MTg2OTg1MjI2" f3durn="urn:adsk.wipprod:dm.lineage:er7lF2gcRpaTRLaYGySQig" pcbguid="eab0e8ed-70a1-480c-828d-d798c72a6244" lastpulledtime="" lastsyncedchangeguid="b07c1c9a-3535-4595-c032-07d5989b0b80"/>
 <plain>
 <wire x1="0" y1="0" x2="26.67" y2="0" width="0" layer="20"/>
@@
 <wire x1="26.67" y1="38.725" x2="0" y2="38.735" width="0" layer="20"/>
 <wire x1="0" y1="38.735" x2="0" y2="0" width="0" layer="20"/>
-<text x="13.589" y="36.322" size="1.778" layer="25" align="bottom-center">EKOMIGACZ</text>
-<text x="13.589" y="34.036" size="1.778" layer="25" align="bottom-center">Paweł Wilczewski</text>
+<text x="13.335" y="36.322" size="1.524" layer="25" align="bottom-center">EKOMIGACZ</text>
+<text x="13.335" y="34.036" size="1.524" layer="25" align="bottom-center">Paweł Wilczewski</text>
+<hole x="3.556" y="8.128" drill="3"/>
+<hole x="23.114" y="8.128" drill="3"/>
+<hole x="23.622" y="35.56" drill="3"/>
+<hole x="3.048" y="35.56" drill="3"/>
 </plain>
 <attributes>
@@
 <attribute name="VALUE" x="6.731" y="19.685" size="1.27" layer="27" ratio="10" rot="R90"/>
 </element>
-<element name="JP2" library="jumper" library_urn="urn:adsk.eagle:library:252" package="JP1" package3d_urn="urn:adsk.eagle:package:15455/1" value="" x="22.225" y="10.795" smashed="yes" rot="R270">
+<element name="JP2" library="jumper" library_urn="urn:adsk.eagle:library:252" package="JP1" package3d_urn="urn:adsk.eagle:package:15455/1" value="" x="22.225" y="15.367" smashed="yes" rot="R270">
 <attribute name="NAME" x="19.685" y="12.446" size="1.27" layer="25" ratio="10"/>
-<attribute name="VALUE" x="19.685" y="7.874" size="1.27" layer="27" ratio="10"/>
+<attribute name="VALUE" x="19.685" y="12.446" size="1.27" layer="27" ratio="10"/>
 </element>
 <element name="LED1" library="led" library_urn="urn:adsk.eagle:library:259" package="LED5MM" package3d_urn="urn:adsk.eagle:package:15799/2" value="" x="22.225" y="22.225" smashed="yes" rot="R180">
@@
 <contactref element="JP2" pad="1"/>
 <contactref element="R3" pad="2"/>
-<wire x1="18.4404" y1="13.4112" x2="18.4404" y2="14.5288" width="0.3048" layer="1"/>
-<wire x1="20.955" y1="10.8966" x2="18.4404" y2="13.4112" width="0.3048" layer="1"/>
-<wire x1="18.4404" y1="14.5288" x2="18.415" y2="14.605" width="0.3048" layer="1"/>
-<wire x1="20.955" y1="10.8966" x2="20.955" y2="10.795" width="0.3048" layer="1"/>
+<wire x1="20.955" y1="15.367" x2="19.177" y2="15.367" width="0.3048" layer="1"/>
+<wire x1="18.415" y1="14.605" x2="19.177" y2="15.367" width="0.3048" layer="1"/>
 </signal>
 <signal name="N$7">
 <contactref element="JP2" pad="2"/>
 <contactref element="LED1" pad="A"/>
-<wire x1="23.4696" y1="10.8966" x2="23.4696" y2="22.0726" width="0.3048" layer="1"/>
+<wire x1="23.4696" y1="15.4686" x2="23.4696" y2="22.0726" width="0.3048" layer="1"/>
 <wire x1="23.4696" y1="22.0726" x2="23.495" y2="22.225" width="0.3048" layer="1"/>
-<wire x1="23.4696" y1="10.8966" x2="23.495" y2="10.795" width="0.3048" layer="1"/>
+<wire x1="23.4696" y1="15.4686" x2="23.495" y2="15.367" width="0.3048" layer="1"/>
 </signal>
 <signal name="N$2">

Commit message: PCB and model update
Parts:
- moved LED1 14.3 mm to (9.78, 15.1), turned to 90 degrees
- moved R2 9.91 mm to (9.78, 29.6)
- moved R3 9.64 mm to (16.4, 23.7), turned to 270 degrees
- moved R1 7.19 mm to (3.17, 23.7), turned to 90 degrees
- moved JP1 7.13 mm to (3.30, 15.1)
- moved JP2 5.85 mm to (16.4, 15.1), turned to 180 degrees
- moved TIMER 3.87 mm to (9.78, 23.7)
- moved X1 3.30 mm to (10.0, 2.92)
- moved C1 3.06 mm to (10.0, 8.51)
Routing:
- net N$4: track 73.2 -> 20.8 mm
- net N$9: track 43.8 -> 21.7 mm
- net 5V: track 8.04 -> 23.4 mm
- net N$7: track 6.86 -> 16.4 mm
- net N$1: track 17.9 -> 9.86 mm
- net N$5: track 40.8 -> 39.6 mm
- net N$6: track 2.86 -> 2.29 mm
Other:
- board size 26.7 x 38.7 mm -> 19.6 x 38.7 mm
